File: PCB/LED Display.sch (EAGLE design)
At the start: 38 parts, among them IC1 LM2596S, IC2 LTC485S, IC3 MEGA32-A, X1 RJ45-6L21-B

Commit message: Fixes for hardware.
Parts:
- +, -, CHANNEL: value DTE6 -> DTS-6; device switch-misc:DTE6 -> switch-tact:DTS-6
Connections:
- net GND: now also +.4, -.4, CHANNEL.4; no longer +.S@1, -.S@1, CHANNEL.S@1
- net N$14: now also -.1; no longer -.P@1
- net N$26: now also +.1; no longer +.P@1
- net N$27: now also CHANNEL.1; no longer CHANNEL.P@1
Changed lines of the file:
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@@
 </part>
 <part name="DISPLAY" library="display-nfd" deviceset="NFD-4631" device=""/>
-<part name="-" library="switch-misc" deviceset="DT" device="E6"/>
-<part name="+" library="switch-misc" deviceset="DT" device="E6"/>
-<part name="CHANNEL" library="switch-misc" deviceset="DT" device="E6"/>
+<part name="-" library="switch-tact" deviceset="DTS-6" device=""/>
+<part name="+" library="switch-tact" deviceset="DTS-6" device=""/>
+<part name="CHANNEL" library="switch-tact" deviceset="DTS-6" device=""/>
 <part name="GND5" library="supply1" deviceset="GND" device=""/>
 <part name="GND6" library="supply1" deviceset="GND" device=""/>
@@
 </instance>
 <instance part="DISPLAY" gate="G$1" x="223.52" y="53.34" rot="R90"/>
-<instance part="-" gate="1" x="256.54" y="45.72" rot="R270"/>
-<instance part="+" gate="1" x="256.54" y="66.04" rot="R270"/>
-<instance part="CHANNEL" gate="1" x="254" y="86.36" rot="R270"/>
+<instance part="-" gate="G$1" x="259.08" y="45.72" rot="R270"/>
+<instance part="+" gate="G$1" x="256.54" y="66.04" rot="R270"/>
+<instance part="CHANNEL" gate="G$1" x="254" y="86.36" rot="R270"/>
 <instance part="GND5" gate="1" x="261.62" y="60.96"/>
-<instance part="GND6" gate="1" x="261.62" y="40.64"/>
+<instance part="GND6" gate="1" x="264.16" y="40.64"/>
 <instance part="GND7" gate="1" x="259.08" y="81.28"/>
 <instance part="R7" gate="G$1" x="182.88" y="55.88"/>
@@
 </segment>
 <segment>
-<pinref part="+" gate="1" pin="S@1"/>
+<pinref part="+" gate="G$1" pin="4"/>
 <pinref part="GND5" gate="1" pin="GND"/>
 </segment>
 <segment>
-<pinref part="-" gate="1" pin="S@1"/>
+<pinref part="-" gate="G$1" pin="4"/>
 <pinref part="GND6" gate="1" pin="GND"/>
 </segment>
 <segment>
-<pinref part="CHANNEL" gate="1" pin="S@1"/>
+<pinref part="CHANNEL" gate="G$1" pin="4"/>
 <pinref part="GND7" gate="1" pin="GND"/>
 </segment>
@@
 <wire x1="170.18" y1="30.48" x2="210.82" y2="30.48" width="0.1524" layer="91"/>
 <wire x1="210.82" y1="30.48" x2="210.82" y2="33.02" width="0.1524" layer="91"/>
-<pinref part="-" gate="1" pin="P@1"/>
 <wire x1="210.82" y1="33.02" x2="251.46" y2="33.02" width="0.1524" layer="91"/>
-<wire x1="251.46" y1="33.02" x2="251.46" y2="43.18" width="0.1524" layer="91"/>
+<pinref part="-" gate="G$1" pin="1"/>
+<wire x1="254" y1="45.72" x2="251.46" y2="45.72" width="0.1524" layer="91"/>
+<wire x1="251.46" y1="45.72" x2="251.46" y2="33.02" width="0.1524" layer="91"/>
 </segment>
 </net>
@@
 <wire x1="208.28" y1="33.02" x2="208.28" y2="35.56" width="0.1524" layer="91"/>
 <wire x1="208.28" y1="35.56" x2="248.92" y2="35.56" width="0.1524" layer="91"/>
-<wire x1="248.92" y1="35.56" x2="248.92" y2="63.5" width="0.1524" layer="91"/>
-<pinref part="+" gate="1" pin="P@1"/>
-<wire x1="248.92" y1="63.5" x2="251.46" y2="63.5" width="0.1524" layer="91"/>
+<wire x1="248.92" y1="35.56" x2="248.92" y2="66.04" width="0.1524" layer="91"/>
+<pinref part="+" gate="G$1" pin="1"/>
+<wire x1="251.46" y1="66.04" x2="248.92" y2="66.04" width="0.1524" layer="91"/>
 </segment>
 </net>
@@
 <wire x1="205.74" y1="35.56" x2="205.74" y2="38.1" width="0.1524" layer="91"/>
 <wire x1="205.74" y1="38.1" x2="246.38" y2="38.1" width="0.1524" layer="91"/>
-<wire x1="246.38" y1="38.1" x2="246.38" y2="83.82" width="0.1524" layer="91"/>
-<pinref part="CHANNEL" gate="1" pin="P@1"/>
-<wire x1="246.38" y1="83.82" x2="248.92" y2="83.82" width="0.1524" layer="91"/>
-</segment>
-</net>
+<wire x1="246.38" y1="38.1" x2="246.38" y2="86.36" width="0.1524" layer="91"/>
+<pinref part="CHANNEL" gate="G$1" pin="1"/>
+<wire x1="248.92" y1="86.36" x2="246.38" y2="86.36" width="0.1524" layer="91"/>
+</segment>
+</net>

Commit message: Numerous fixes.
Parts:
- removed DMX: DMX, pinhead:PINHD-1X3
- removed POWER: 7-40V, pinhead:PINHD-1X2
- added X2: (no value), con-wago-508:W237-02P
- added X3: (no value), con-wago-508:W237-03P
Connections:
- net GND: now also X2-2.KL, X3-3.KL; no longer DMX.3, POWER.1
- net N$10: now also X3-1.KL; no longer DMX.1
- net N$14: now also +.1; no longer -.1
- net N$26: now also -.1; no longer +.1
- net N$41: now also X2-1.KL; no longer POWER.2
- net N$9: now also X3-2.KL; no longer DMX.2
Other:
- moved on the sheet: +, -
Changed lines of the file:
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@@
 <parts>
 <part name="IC1" library="national-semiconductor" deviceset="LM2596" device="S"/>
-<part name="POWER" library="pinhead" deviceset="PINHD-1X2" device="" value="7-40V"/>
 <part name="R1" library="resistor" deviceset="R-EU_" device="M0805" value="3k09">
 <attribute name="FARNEL" value="2502845"/>
@@
 <attribute name="FARNEL" value="2101194"/>
 </part>
-<part name="DMX" library="pinhead" deviceset="PINHD-1X3" device="" value="DMX"/>
 <part name="IC2" library="linear-technology" deviceset="LTC485" device="S">
 <attribute name="OC_FARNELL" value="1564306"/>
@@
 </part>
 <part name="DISPLAY" library="display-nfd" deviceset="NFD-4631" device=""/>
+<part name="+" library="switch-tact" deviceset="DTS-6" device=""/>
 <part name="-" library="switch-tact" deviceset="DTS-6" device=""/>
-<part name="+" library="switch-tact" deviceset="DTS-6" device=""/>
 <part name="CHANNEL" library="switch-tact" deviceset="DTS-6" device=""/>
 <part name="GND5" library="supply1" deviceset="GND" device=""/>
@@
 <part name="X1" library="con-tycoelectronics" deviceset="RJ45*2" device="1-B" technology="-6L"/>
 <part name="R6" library="resistor" deviceset="R-EU_" device="M0805" value="470"/>
+<part name="X2" library="con-wago-508" deviceset="W237-02P" device=""/>
+<part name="X3" library="con-wago-508" deviceset="W237-03P" device=""/>
 </parts>
 <sheets>
@@
 <instances>
 <instance part="IC1" gate="G$1" x="30.48" y="66.04"/>
-<instance part="POWER" gate="G$1" x="-10.16" y="71.12" rot="R180"/>
 <instance part="R1" gate="G$1" x="91.44" y="66.04" rot="R90">
 <attribute name="FARNEL" x="91.44" y="66.04" size="1.778" layer="96" rot="R90" display="off"/>
@@
 <attribute name="FARNEL" x="48.26" y="55.88" size="1.778" layer="96" rot="R90" display="off"/>
 </instance>
-<instance part="DMX" gate="A" x="266.7" y="17.78"/>
 <instance part="IC2" gate="G$1" x="205.74" y="20.32"/>
 <instance part="GND2" gate="1" x="215.9" y="10.16"/>
@@
 </instance>
 <instance part="DISPLAY" gate="G$1" x="223.52" y="53.34" rot="R90"/>
-<instance part="-" gate="G$1" x="259.08" y="45.72" rot="R270"/>
-<instance part="+" gate="G$1" x="256.54" y="66.04" rot="R270"/>
+<instance part="+" gate="G$1" x="259.08" y="45.72" rot="R270"/>
+<instance part="-" gate="G$1" x="256.54" y="66.04" rot="R270"/>
 <instance part="CHANNEL" gate="G$1" x="254" y="86.36" rot="R270"/>
 <instance part="GND5" gate="1" x="261.62" y="60.96"/>
@@
 <instance part="X1" gate="G$1" x="284.48" y="17.78"/>
 <instance part="R6" gate="G$1" x="182.88" y="58.42"/>
+<instance part="X2" gate="-1" x="-10.16" y="71.12"/>
+<instance part="X2" gate="-2" x="-10.16" y="68.58"/>
+<instance part="X3" gate="-1" x="269.24" y="20.32" rot="R180"/>
+<instance part="X3" gate="-2" x="269.24" y="17.78" rot="R180"/>
+<instance part="X3" gate="-3" x="269.24" y="15.24" rot="R180"/>
 </instances>
 <busses>
@@
 <net name="GND" class="0">
 <segment>
-<pinref part="POWER" gate="G$1" pin="1"/>
-<wire x1="-7.62" y1="68.58" x2="0" y2="68.58" width="0.1524" layer="91"/>
+<wire x1="-5.08" y1="68.58" x2="0" y2="68.58" width="0.1524" layer="91"/>
 <wire x1="0" y1="68.58" x2="0" y2="60.96" width="0.1524" layer="91"/>
 <pinref part="IC1" gate="G$1" pin="GND"/>
@@
 <wire x1="48.26" y1="48.26" x2="48.26" y2="53.34" width="0.1524" layer="91"/>
 <junction x="48.26" y="48.26"/>
+<pinref part="X2" gate="-2" pin="KL"/>
 </segment>
 <segment>
@@
 <pinref part="GND2" gate="1" pin="GND"/>
 <wire x1="215.9" y1="12.7" x2="215.9" y2="15.24" width="0.1524" layer="91"/>
-<pinref part="DMX" gate="A" pin="3"/>
 <wire x1="215.9" y1="15.24" x2="228.6" y2="15.24" width="0.1524" layer="91"/>
 <junction x="215.9" y="15.24"/>
@@
 <pinref part="X1" gate="G$1" pin="S@3"/>
 <junction x="284.48" y="5.08"/>
+<pinref part="X3" gate="-3" pin="KL"/>
 </segment>
 <segment>
@@
 </segment>
 <segment>
+<pinref part="-" gate="G$1" pin="4"/>
+<pinref part="GND5" gate="1" pin="GND"/>
+</segment>
+<segment>
 <pinref part="+" gate="G$1" pin="4"/>
-<pinref part="GND5" gate="1" pin="GND"/>
-</segment>
-<segment>
-<pinref part="-" gate="G$1" pin="4"/>
 <pinref part="GND6" gate="1" pin="GND"/>
 </segment>
@@
 <net name="N$9" class="0">
 <segment>
-<pinref part="DMX" gate="A" pin="2"/>
 <pinref part="R4" gate="G$1" pin="1"/>
 <wire x1="264.16" y1="17.78" x2="259.08" y2="17.78" width="0.1524" layer="91"/>
@@
 <wire x1="259.08" y1="25.4" x2="259.08" y2="17.78" width="0.1524" layer="91"/>
 <junction x="259.08" y="17.78"/>
+<pinref part="X3" gate="-2" pin="KL"/>
 </segment>
 </net>
 <net name="N$10" class="0">
 <segment>
-<pinref part="DMX" gate="A" pin="1"/>
 <pinref part="R5" gate="G$1" pin="1"/>
 <wire x1="264.16" y1="20.32" x2="256.54" y2="20.32" width="0.1524" layer="91"/>
@@
 <wire x1="256.54" y1="27.94" x2="256.54" y2="20.32" width="0.1524" layer="91"/>
 <junction x="256.54" y="20.32"/>
+<pinref part="X3" gate="-1" pin="KL"/>
 </segment>
 </net>
@@
 <wire x1="210.82" y1="30.48" x2="210.82" y2="33.02" width="0.1524" layer="91"/>
 <wire x1="210.82" y1="33.02" x2="251.46" y2="33.02" width="0.1524" layer="91"/>
-<pinref part="-" gate="G$1" pin="1"/>
+<pinref part="+" gate="G$1" pin="1"/>
 <wire x1="254" y1="45.72" x2="251.46" y2="45.72" width="0.1524" layer="91"/>
 <wire x1="251.46" y1="45.72" x2="251.46" y2="33.02" width="0.1524" layer="91"/>
@@
 <wire x1="208.28" y1="35.56" x2="248.92" y2="35.56" width="0.1524" layer="91"/>
 <wire x1="248.92" y1="35.56" x2="248.92" y2="66.04" width="0.1524" layer="91"/>
-<pinref part="+" gate="G$1" pin="1"/>
+<pinref part="-" gate="G$1" pin="1"/>
 <wire x1="251.46" y1="66.04" x2="248.92" y2="66.04" width="0.1524" layer="91"/>
 </segment>
@@
 <net name="N$41" class="0">
 <segment>
-<pinref part="POWER" gate="G$1" pin="2"/>
 <pinref part="D3" gate="G$1" pin="A"/>
-<wire x1="-7.62" y1="71.12" x2="0" y2="71.12" width="0.1524" layer="91"/>
-</segment>
-</net>
+<wire x1="-5.08" y1="71.12" x2="0" y2="71.12" width="0.1524" layer="91"/>
+<pinref part="X2" gate="-1" pin="KL"/>
+</segment>
+</net>
