File: PCB/LED Display.brd (EAGLE design)
At the start: 64.5 x 42.8 mm, 38 parts, among them IC1 LM2596S, IC2 LTC485S, IC3 MEGA32-A, X1 RJ45-6L21-B

Commit message: Fixes for hardware.
Parts:
- +, -, CHANNEL: value DTE6 -> DTS-6; device switch-misc:DTE6 -> switch-tact:DTS-6
- moved R12 1.09 mm to (50.9, 38.1)
- moved C3 1.09 mm to (53.2, 38.1)
- moved LED1 0.90 mm to (58.3, 38.7)
- moved R7 0.76 mm to (52.6, 31.5)
- moved R8 0.76 mm to (52.6, 26.2)
- moved U$3 0.25 mm to (1.65, 30.9)
- moved DMX 0.13 mm to (5.46, 9.91)
- turned + to 90 degrees
- turned - to 90 degrees
- turned CHANNEL to 90 degrees
Connections:
- net GND: now also +.4, -.4, CHANNEL.4; no longer +.2, -.2, CHANNEL.2
- net N$14: now also -.1; no longer -.4
- net N$26: now also +.1; no longer +.4
- net N$27: now also CHANNEL.1; no longer CHANNEL.4
Routing:
- net GND: track 0.51 -> 17.1 mm, vias 14 -> 13
- net N$31: track 42.1 -> 44.0 mm
- net DI: track 59.7 -> 61.2 mm
- net N$16: track 17.8 -> 16.7 mm
- net N$20: track 18.5 -> 19.2 mm
- net N$26: track 31.3 -> 31.8 mm
- added copper zone on layer 1, net N$13
- added copper zone on layer 1, net N$25
- added copper zone on layer 1, net N$28
Other:
- board size 64.5 x 42.8 mm -> 62 x 42.5 mm
- board text added: "-"
- board text added: "Mode"

Commit message: Numerous fixes.
Parts:
- removed DMX: DMX, pinhead:1X03
- removed POWER: 7-40V, pinhead:1X02
- added X2: (no value), con-wago-508:W237-132
- added X3: (no value), con-wago-508:W237-133
- moved - 11.6 mm to (58.5, 18.9)
- moved + 9.65 mm to (58.5, 28.7)
- moved C3 7.05 mm to (59.7, 40.9), turned to 0 degrees
- moved D3 3.77 mm to (15.6, 24.5), turned to 270 degrees
- moved R12 3.23 mm to (53.2, 35.8)
- moved U$1 2.57 mm to (22.6, 19.2)
- moved LED1 2.29 mm to (58.4, 36.4)
- moved DISPLAY 2.29 mm to (40.4, 33.0)
- moved R1 2.17 mm to (22.4, 24.9)
- moved C2 2.07 mm to (31.2, 17.4)
- moved R2 2.05 mm to (26.4, 24.9)
- moved R6 1.94 mm to (37.0, 20.2)
- moved R5 1.89 mm to (19.2, 6.10)
- moved R4 1.78 mm to (19.2, 2.16)
- moved JP2 1.69 mm to (40.8, 1.91)
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Connections:
- net GND: now also X2.2, X3.3; no longer DMX.3, POWER.1
- net N$10: now also X3.1; no longer DMX.1
- net N$14: now also +.1; no longer -.1
- net N$26: now also -.1; no longer +.1
- net N$41: now also X2.1; no longer POWER.2
- net N$9: now also X3.2; no longer DMX.2
Routing:
- net N$16: track 16.7 -> 29.2 mm
- net PA7: track 58.4 -> 65.5 mm
- net PA6: track 56.8 -> 63.6 mm
- net DI: track 61.2 -> 54.6 mm
- net N$9: track 25.1 -> 19.0 mm
- net N$21: track 29.3 -> 23.2 mm
- net PA5: track 56.1 -> 61.8 mm
- net N$14: track 45.3 -> 40.2 mm
- net N$10: track 21.0 -> 16.7 mm
- net PA4: track 56.5 -> 60.4 mm
- net N$26: track 31.8 -> 28.2 mm
- net N$5: track 8.28 -> 11.6 mm
- net +5V: track 189.5 -> 186.4 mm
- net N$31: track 44.0 -> 40.9 mm
- net N$2: track 9.35 -> 12.0 mm
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Other:
- board text removed: "2017"

Commit message: Tidy the board.
Parts:
- moved R12 6.36 mm to (53.6, 29.5)
- moved R7 6.36 mm to (53.6, 25.1)
- moved R8 5.09 mm to (53.6, 20.7)
Routing:
- net N$31: track 40.9 -> 33.8 mm
- net N$35: track 25.0 -> 18.4 mm
- net N$21: track 23.2 -> 29.3 mm
- net N$29: track 19.7 -> 14.5 mm
- net N$20: track 17.7 -> 22.7 mm
- net N$16: track 29.2 -> 33.8 mm
- net +5V: track 186.4 -> 189.3 mm
- net N$22: track 25.3 -> 23.7 mm
- net N$24: track 33.3 -> 32.2 mm
- net N$23: track 40.9 -> 40.2 mm
- net N$32: track 29.8 -> 29.3 mm
